File: Periphery.kicad_sch (KiCad schematic)
At the start: 10 parts, among them SW1 Mitsumi R-667996, SW2 Mitsumi R-667996, U2 IS31FL3726A-QFLS4, U3 THVD1420DRLR

Commit message: Started power protection hotswap circuit
Parts:
- added U4: RS31340B, custom_Power_QFN:QFN-10-1EP_2x2mm_P0.5mm, symbol custom_Power_Management:RS31340
Connections:
- net GND: now also U4.8 (GND), U4.GND
- net NRST: now also U4.3 (PG)
- net VDD: now also U4.6 (OUT)
- new net VBUS: U4.5 (IN)
- no-connect marks 1 -> 2
Other:
- note added: "Enables after power is stable"
