File: ESP32-S3 Hub.kicad_pcb (KiCad board)
At the start: 6 copper layers, 15 x 30 mm, 73 parts, among them J1 Precidip 853-87-004-20-001101, J10 Precidip 853-87-004-20-001101, J11 FPC 0.3mm Aces 51688-0070M, J12 Precidip 853-87-004-20-001101, J13 TE 3-2363961-0 receptacle, J15 Precidip 853-87-004-20-001101, J16 TE 3-2363961-0 receptacle, J18 Precidip 852-10-004-20-001101, J2 Precidip 853-87-004-20-001101, J3 FPC 0.3mm Aces 51688-0070M, J4 Precidip 853-87-004-20-001101, J5 FPC 0.3mm Aces 51688-0070M, J6 Precidip 853-87-004-20-001101, J7 Precidip 853-87-004-20-001101, J8 FPC 0.3mm Aces 51688-0070M, J9 Precidip 853-87-004-20-001101, SW1 Mitsumi R-667996, SW2 Mitsumi R-667996, U1 ESP32-S3 FN8, U2 SN74LV595A, U3 THVD1420DRLR, U4 TPS2521ARPWR, U5 SN74LV595A, U6 TS5A3159DCK, Y1 2 pin 40MHZ, 10ppm tol., 20pp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

Commit message: Changed i2c resistors to be stronger
The distance is really short and I was only ever planning on having a few devices per hub, so strength is increased.
Parts:
- R8, R9: value 10k -> 2.2k
Changed lines of the file:
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@@
 			)
 		)
-		(property "Value" "10k"
+		(property "Value" "2.2k"
 			(at 0 1.17 90)
 			(layer "F.Fab")
@@
 			)
 		)
-		(property "LCSC" "C25744"
+		(property "LCSC" "C25879"
 			(at 0 0 90)
 			(unlocked yes)
@@
 			)
 		)
-		(property "Value" "10k"
+		(property "Value" "2.2k"
 			(at 0 1.17 90)
 			(layer "F.Fab")
@@
 			)
 		)
-		(property "LCSC" "C25744"
+		(property "LCSC" "C25879"
 			(at 0 0 0)
 			(layer "F.SilkS")
